Commit message: feat(sim): add T-0 lidar and rasterized Nav2 map for wall avoidance
Mount a 360° GPU lidar on T-0, bridge /scan to Nav2 obstacle layers, and
rasterize furnished interior collision boxes into the escape-room occupancy map.

Co-authored-by: Cursor <cursoragent@cursor.com>

File: examples/meshes/escape_room/gazebo/models/t0_robot/t0_robot.urdf (robot description, URDF)
Before this commit: robot t0_robot, 4 links, 3 joints
Links:
- added link laser_link
Joints:
- added joint laser_joint: type fixed, parent base_link, child laser_link, origin xyz=0.12 0 0.06 rpy=0 0 0
